Commit message: 🦄 refactor(config):
add rs into urdf and bringup

File: src/xtark_description/urdf/xtark_description.urdf (robot description, URDF)
Before this commit: robot xtark_description, 10 links, 9 joints
Joints:
- joint camera_joint: origin xyz=0.21091 0 0.17748 rpy=0 -0.34907 0 -> xyz=0.11 0 0.8802 rpy=0 0 0

Commit message: ✨ feat(depth camera): switch to gemini

File: src/xtark_description/urdf/xtark_description.urdf (robot description, URDF)
Before this commit: robot xtark_description, 10 links, 9 joints
Joints:
- joint camera_joint: origin xyz=0.11 0 0.8802 rpy=0 0 0 -> xyz=0.1 0.105 0.8802 rpy=0 0 0
